Commit message: localization y navigation

File: limo_description/urdf/limo_ackerman.xacro (robot description, xacro)
@@ -1,4 +1,5 @@
 <?xml version="1.0"?>
 <robot name="limo_ackerman" xmlns:xacro="http://ros.org/wiki/xacro">
+    <xacro:arg name="robot_namespace" default="/" />
     <xacro:include filename="$(find uned_limo_gazebo)/limo_description/urdf/limo_xacro.xacro" />
     <xacro:include filename="$(find uned_limo_gazebo)/limo_description/urdf/limo_steering_hinge.xacro" />
@@ -16,12 +17,12 @@
     <xacro:property name="wheel_length" value="0.045" />
     <xacro:property name="wheel_radius" value="0.045" />
-    <link name="$(arg robot_namespace)base_footprint"/>
-    <joint name="$(arg robot_namespace)base_joint" type="fixed">
-        <parent link="$(arg robot_namespace)base_footprint"/>
-        <child link="$(arg robot_namespace)base_link"/>
+    <link name="base_footprint"/>
+    <joint name="base_joint" type="fixed">
+        <parent link="base_footprint"/>
+        <child link="base_link"/>
         <origin xyz="0.0 0.0 0.15" rpy="0 0 0"/>
     </joint>
     <!-- Base link -->
-    <link name="$(arg robot_namespace)base_link">
+    <link name="base_link">
         <visual>
             <origin xyz="0 0 -0.15" rpy="0 0 1.57" />
@@ -37,5 +38,5 @@
         </collision>
     </link>
-    <link name="$(arg robot_namespace)inertial_link">
+    <link name="inertial_link">
         <inertial>
             <origin xyz="0.0 0.0 0.0" />
@@ -46,8 +47,8 @@
         </inertial>
     </link>
-    <joint name="$(arg robot_namespace)inertial_joint" type="fixed">
+    <joint name="inertial_joint" type="fixed">
         <origin xyz="0 0 0" rpy="0 0 0" />
-        <parent link="$(arg robot_namespace)base_link" />
-        <child link="$(arg robot_namespace)inertial_link" />
+        <parent link="base_link" />
+        <child link="inertial_link" />
     </joint>
     <xacro:limo_laser parent_prefix="base_link" frame_prefix="laser">
@@ -66,5 +67,5 @@
         <origin xyz="${wheelbase/2} ${-track/2} ${wheel_vertical_offset}" rpy="${M_PI} 0 0" />
     </xacro:limo_right_steering_hinge>
-    <link name="$(arg robot_namespace)rear_left_wheel_link">
+    <link name="rear_left_wheel_link">
         <inertial>
             <origin xyz="0 0 0" />
@@ -85,11 +86,15 @@
         </collision>
     </link>
-    <joint name="$(arg robot_namespace)rear_left_wheel" type="continuous">
-        <parent link="$(arg robot_namespace)base_link"/>
-        <child link="$(arg robot_namespace)rear_left_wheel_link"/>
+    <joint name="rear_left_wheel" type="continuous">
+        <parent link="base_link"/>
+        <child link="rear_left_wheel_link"/>
         <origin xyz="${-wheelbase/2} ${track/2} ${wheel_vertical_offset}" rpy="0 0 0" />
-        <axis xyz="0 1 0"/>
+        <axis xyz="0 1 0">
+            <limit>
+                <effort>50</effort>  <!-- from Gazebo Classic <torque> diff plugin -->
+            </limit>
+        </axis>
     </joint>
-    <link name="$(arg robot_namespace)rear_right_wheel_link">
+    <link name="rear_right_wheel_link">
         <inertial>
             <origin xyz="0 0 0" />
@@ -110,9 +115,13 @@
             </collision>
         </link>
-        <joint name="$(arg robot_namespace)rear_right_wheel" type="continuous">
-            <parent link="$(arg robot_namespace)base_link"/>
-            <child link="$(arg robot_namespace)rear_right_wheel_link"/>
+        <joint name="rear_right_wheel" type="continuous">
+            <parent link="base_link"/>
+            <child link="rear_right_wheel_link"/>
             <origin xyz="${-wheelbase/2} ${-track/2} ${wheel_vertical_offset}" rpy="${M_PI} 0 0" />
-            <axis xyz="0 -1 0"/>
+            <axis xyz="0 -1 0">
+                <limit>
+                    <effort>50</effort>  <!-- from Gazebo Classic <torque> diff plugin -->
+                </limit>
+            </axis>
         </joint>
 </robot>

File: limo_description/urdf/limo_four_diff.xacro (robot description, xacro)
@@ -15,12 +15,12 @@
     <xacro:property name="wheel_length" value="0.045" />
     <xacro:property name="wheel_radius" value="0.045" />
-  <link name="$(arg robot_namespace)base_footprint"/>
-  <joint name="$(arg robot_namespace)base_joint" type="fixed">
-    <parent link="$(arg robot_namespace)base_footprint"/>
-    <child link="$(arg robot_namespace)base_link"/>
-    <origin xyz="0.0 0.0 0.15" rpy="0 0 0"/>
-  </joint>
+    <link name="base_footprint"/>
+    <joint name="base_joint" type="fixed">
+      <parent link="base_footprint"/>
+      <child link="base_link"/>
+      <origin xyz="0.0 0.0 0.15" rpy="0 0 0"/>
+    </joint>
     <!-- Base link -->
-    <link name="$(arg robot_namespace)base_link">
+    <link name="base_link">
         <visual>
             <origin xyz="0 0 -0.15" rpy="0 0 1.57" />
@@ -37,5 +37,5 @@
         </collision>
     </link>
-    <link name="$(arg robot_namespace)inertial_link">
+    <link name="inertial_link">
         <inertial>
             <origin xyz="0.0 0.0 0.0" />
@@ -46,8 +46,8 @@
         </inertial>
     </link>
-    <joint name="$(arg robot_namespace)inertial_joint" type="fixed">
+    <joint name="inertial_joint" type="fixed">
         <origin xyz="0 0 0" rpy="0 0 0" />
-        <parent link="$(arg robot_namespace)base_link" />
-        <child link="$(arg robot_namespace)inertial_link" />
+        <parent link="base_link" />
+        <child link="inertial_link" />
     </joint>
     <xacro:limo_laser parent_prefix="base_link" frame_prefix="laser">

File: limo_description/urdf/limo_steering_hinge.xacro (robot description, xacro)
@@ -1,6 +1,6 @@
 <?xml version="1.0"?>
-<robot xmlns:xacro="http://ros.org/wiki/xacro">
+<robot name="limo_steering_hinge" xmlns:xacro="http://ros.org/wiki/xacro">
     <xacro:macro name="limo_left_steering_hinge" params="parent_prefix wheel_prefix *joint_pose">
-        <link name="$(arg robot_namespace)${wheel_prefix}">
+        <link name="${wheel_prefix}">
             <inertial>
               <mass value="0.25" />
@@ -21,7 +21,7 @@
             </collision>
         </link>
-        <joint name="$(arg robot_namespace)${wheel_prefix}_wheel" type="revolute">
-            <parent link="$(arg robot_namespace)${parent_prefix}"/>
-            <child link="$(arg robot_namespace)${wheel_prefix}"/>
+        <joint name="${wheel_prefix}_wheel" type="revolute">
+            <parent link="${parent_prefix}"/>
+            <child link="${wheel_prefix}"/>
             <xacro:insert_block name="joint_pose"/>
             <axis xyz="0 0 1" />
@@ -29,5 +29,5 @@
             <dynamics damping="1.0" friction="2.0"/>
         </joint>
-        <link name="$(arg robot_namespace)front_left_wheel_link">
+        <link name="front_left_wheel_link">
           <inertial>
             <mass value="0.25" />
@@ -38,5 +38,5 @@
               <origin xyz="0 0 0" rpy="0 0 0" />
               <geometry>
-                  <mesh filename="file://$(find uned_limo_gazebo)/limo_description/meshes/limo_optimal_wheels.dae" scale="1 1 1"/>
+                  <mesh filename="file://$(find uned_limo_gazebo)/limo_description/meshes/limo_optimal_wheels.dae" />
               </geometry>
           </visual>
@@ -48,7 +48,7 @@
           </collision>
       </link>
-      <joint name="$(arg robot_namespace)front_left_wheel" type="continuous">
-          <parent link="$(arg robot_namespace)${wheel_prefix}"/>
-          <child link="$(arg robot_namespace)front_left_wheel_link"/>
+      <joint name="front_left_wheel" type="continuous">
+          <parent link="${wheel_prefix}"/>
+          <child link="front_left_wheel_link"/>
           <origin xyz="0 0 0" rpy="0 0  0" />
           <axis xyz="0 1 0"/>
@@ -56,5 +56,5 @@
     </xacro:macro>
     <xacro:macro name="limo_right_steering_hinge" params="parent_prefix wheel_prefix *joint_pose">
-        <link name="$(arg robot_namespace)${wheel_prefix}">
+        <link name="${wheel_prefix}">
           <inertial>
             <mass value="0.25" />
@@ -75,7 +75,7 @@
             </collision>
         </link>
-        <joint name="$(arg robot_namespace)${wheel_prefix}_wheel" type="revolute">
-            <parent link="$(arg robot_namespace)${parent_prefix}"/>
-            <child link="$(arg robot_namespace)${wheel_prefix}"/>
+        <joint name="${wheel_prefix}_wheel" type="revolute">
+            <parent link="${parent_prefix}"/>
+            <child link="${wheel_prefix}"/>
             <xacro:insert_block name="joint_pose"/>
             <axis xyz="0 0 -1"/>
@@ -83,5 +83,5 @@
             <dynamics damping="1.0" friction="2.0"/>
         </joint>
-        <link name="$(arg robot_namespace)front_right_wheel_link">
+        <link name="front_right_wheel_link">
           <inertial>
             <mass value="0.25" />
@@ -92,5 +92,5 @@
               <origin xyz="0 0 0" rpy="0 0 0" />
               <geometry>
-                  <mesh filename="file://$(find uned_limo_gazebo)/limo_description/meshes/limo_optimal_wheels.dae" scale="1 1 1" />
+                  <mesh filename="file://$(find uned_limo_gazebo)/limo_description/meshes/limo_optimal_wheels.dae" />
               </geometry>
           </visual>
@@ -102,8 +102,8 @@
           </collision>
       </link>
-      <joint name="$(arg robot_namespace)front_right_wheel" type="continuous">
-          <parent link="$(arg robot_namespace)${wheel_prefix}"/>
-          <child link="$(arg robot_namespace)front_right_wheel_link"/>
-          <origin xyz="0 0 0" rpy="0 0  0" />
+      <joint name="front_right_wheel" type="continuous">
+          <parent link="${wheel_prefix}"/>
+          <child link="front_right_wheel_link"/>
+          <origin xyz="0 0 0" rpy="0 0 0" />
           <axis xyz="0 -1 0"/>
       </joint>

File: limo_description/urdf/limo_xacro.xacro (robot description, xacro)
@@ -1,7 +1,7 @@
 <?xml version="1.0"?>
-<robot xmlns:xacro="http://ros.org/wiki/xacro">
+<robot name="limo_xacro" xmlns:xacro="http://ros.org/wiki/xacro">
     <xacro:include filename="$(find uned_limo_gazebo)/limo_description/urdf/limo_materials.xacro" />
     <xacro:macro name="limo_wheel" params="parent_prefix wheel_prefix reflect *joint_pose">
-        <link name="$(arg robot_namespace)${wheel_prefix}_wheel_link">
+        <link name="${wheel_prefix}_wheel_link">
             <inertial>
                 <origin xyz="0 0 0" />
@@ -12,5 +12,5 @@
                 <origin xyz="0 0 0" rpy="0 0 0" />
                 <geometry>
-                    <mesh filename="file://$(find uned_limo_gazebo)/limo_description/meshes/limo_optimal_wheels.dae" scale="1 1 1"/>
+                    <mesh filename="file://$(find uned_limo_gazebo)/limo_description/meshes/limo_optimal_wheels.dae" />
                 </geometry>
             </visual>
@@ -22,7 +22,7 @@
             </collision>
         </link>
-        <joint name="$(arg robot_namespace)${wheel_prefix}_wheel" type="continuous">
-            <parent link="$(arg robot_namespace)${parent_prefix}"/>
-            <child link="$(arg robot_namespace)${wheel_prefix}_wheel_link"/>
+        <joint name="${wheel_prefix}_wheel" type="continuous">
+            <parent link="${parent_prefix}"/>
+            <child link="${wheel_prefix}_wheel_link"/>
             <xacro:insert_block name="joint_pose"/>
             <axis xyz="0 ${reflect*1} 0">
@@ -34,5 +34,5 @@
     </xacro:macro>
     <xacro:macro name="limo_laser" params="parent_prefix frame_prefix *joint_pose">
-        <link name='$(arg robot_namespace)${frame_prefix}_link'>
+        <link name='${frame_prefix}_link'>
             <pose>0 0 0 0 0 0</pose>
             <inertial>
@@ -59,12 +59,12 @@
             </collision>
         </link>
-        <joint type="fixed" name="$(arg robot_namespace)laser_joint">
+        <joint type="fixed" name="laser_joint">
             <xacro:insert_block name="joint_pose"/>
-            <child link="$(arg robot_namespace)${frame_prefix}_link"/>
-            <parent link="$(arg robot_namespace)${parent_prefix}"/>
+            <child link="${frame_prefix}_link"/>
+            <parent link="${parent_prefix}"/>
         </joint>
     </xacro:macro>
     <xacro:macro name="limo_depth_camera" params="parent_prefix frame_prefix *joint_pose">
-        <link name='$(arg robot_namespace)${frame_prefix}_link'>
+        <link name='${frame_prefix}_link'>
             <pose>0 0 0 0 0 0</pose>
             <inertial>
@@ -91,18 +91,18 @@
             </collision>
         </link>
-        <joint type="fixed" name="$(arg robot_namespace)depth_camera_joint">
+        <joint type="fixed" name="depth_camera_joint">
             <xacro:insert_block name="joint_pose"/>
-            <child link="$(arg robot_namespace)${frame_prefix}_link"/>
-            <parent link="$(arg robot_namespace)${parent_prefix}"/>
+            <child link="${frame_prefix}_link"/>
+            <parent link="${parent_prefix}"/>
         </joint>
-        <link name="$(arg robot_namespace)depth_link"></link>
-        <joint name="$(arg robot_namespace)${frame_prefix}_to_camera_joint" type="fixed">
+        <link name="depth_link"></link>
+        <joint name="${frame_prefix}_to_camera_joint" type="fixed">
             <origin xyz="0 0 0" rpy="${-M_PI/2} 0 ${-M_PI/2} "/>
-            <parent link="$(arg robot_namespace)${frame_prefix}_link"/>
-            <child link="$(arg robot_namespace)depth_link"/>
+            <parent link="${frame_prefix}_link"/>
+            <child link="depth_link"/>
         </joint>
     </xacro:macro>
     <xacro:macro name="limo_imu" params="parent_prefix frame_prefix  *joint_pose">
-        <link name='$(arg robot_namespace)${frame_prefix}_link'>
+        <link name='${frame_prefix}_link'>
             <pose>0 0 0 0 0 0</pose>
             <inertial>
@@ -129,8 +129,8 @@
             </collision>
         </link>
-        <joint type="fixed" name="$(arg robot_namespace)imu_joint">
+        <joint type="fixed" name="imu_joint">
             <xacro:insert_block name="joint_pose"/>
-            <child link="$(arg robot_namespace)${frame_prefix}_link"/>
-            <parent link="$(arg robot_namespace)${parent_prefix}"/>
+            <child link="${frame_prefix}_link"/>
+            <parent link="${parent_prefix}"/>
         </joint>
     </xacro:macro>
